File: RGBW Led Driver.kicad_pcb (KiCad board)
At the start: 2 copper layers, 66 x 50.8 mm, 23 parts, among them J1 Screw_Terminal_01x06, Q1 IRLZ44N, Q2 IRLZ44N, Q3 IRLZ44N, Q4 IRLZ44N, U1 TC4427xOA, U2 TC4427xOA

Commit message: Moved global custom libraries locally
Parts:
- D1: footprint custom:ESP32-C6 Supermini -> Custom:ESP32-C6 Supermini
Changed lines of the file:
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@@
 		)
 	)
-	(footprint "custom:ESP32-C6 Supermini"
+	(footprint "Custom:ESP32-C6 Supermini"
 		(layer "F.Cu")
 		(at 182.88 90.22)
@@
 		)
 		(embedded_fonts no)
-		(model "/home/morels/varie/kicad/3d-models/super_mini_esp32_c6_nologo.step"
+		(model "${KIPRJMOD}/libraries/3d-models/super_mini_esp32-c6.step"
 			(offset
 				(xyz 0 13 1.5)
@@
 			)
 			(rotate
-				(xyz 0 0 0)
-			)
-		)
+				(xyz -0 -0 -0)
+			)
+		)

Commit message: Added title
Other:
- board text added: "Claudio M. 2026-10-16"
- board text added: "RGBW Led Driver Rev 0.1^n"
- board text removed: "Claudio M. 2026-10-15"
- board text removed: "Rev 0.1^n"
Changed lines of the file:
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@@
 		(layer "Edge.Cuts")
 	)
-	(gr_text "Rev 0.1^n"
-		(at 160.02 81.28 0)
+	(gr_text "RGBW Led Driver\nRev 0.1^n"
+		(at 156.73865 80.434449 0)
 		(layer "F.SilkS")
 		(effects
 			(font
-				(size 1.5 1.5)
+				(size 1.4 1.4)
 				(thickness 0.3)
 				(bold yes)
@@
 		)
 	)
-	(gr_text "Claudio M.\n2026-10-15"
+	(gr_text "Claudio M.\n2026-10-16"
 		(at 177.821914 123.200256 0)
 		(layer "F.SilkS")

Commit message: Changed from M2 to M3 mounting holes
Parts:
- removed the REF** at (170.2, 80.0)
- removed the REF** at (189.2, 123.2)
- removed the REF** at (130.8, 123.2)
- removed the REF** at (130.8, 80.0)
- added REF**: MountingHole_3.2mm_M3, MountingHole:MountingHole_3.2mm_M3, F.Cu at (189.2, 123.2)
- added REF**: MountingHole_3.2mm_M3, MountingHole:MountingHole_3.2mm_M3, F.Cu at (170.2, 80.0)
- added REF**: MountingHole_3.2mm_M3, MountingHole:MountingHole_3.2mm_M3, F.Cu at (130.8, 123.2)
- added REF**: MountingHole_3.2mm_M3, MountingHole:MountingHole_3.2mm_M3, F.Cu at (130.8, 80.0)
