File: RGBW Led Driver.kicad_pcb (KiCad board)
At the start: 2 copper layers, 66 x 50.8 mm, 23 parts, among them J1 Screw_Terminal_01x06, Q1 IRLZ44N, Q2 IRLZ44N, Q3 IRLZ44N, Q4 IRLZ44N, U1 TC4427xOA, U2 TC4427xOA

Commit message: Switched 4 resistors from vertical to horizontal
Parts:
- R5, R6, R7, R8: footprint Resistor_THT:R_Axial_DIN0207_L6.3mm_D2.5mm_P2.54mm_Vertical -> Resistor_THT:R_Axial_DIN0207_L6.3mm_D2.5mm_P7.62mm_Horizontal
Routing:
- net GND: track 257.7 -> 295.9 mm
- net 5v: track 123.2 -> 124.2 mm
